Commit message: Sim: adopt CAD export (5) — ROS frames, sensor frames, re-solved limits
- fix_urdf.py: root link -> base_link, strip robot name; limits now come
  from joint_limits_from_urdf.py, which solves the closed loop in the URDF
  itself (CAD re-exports change joint local frames)
- make_simple_urdf.py: no 90 deg rotation (CAD is +x forward now), origin at
  hip midpoint, real body COM, shank inertia rotated into body frame, carrier
  COM calibrated to CAD total COM (-7.9 mm), imu_link/gps_link/laser/
  camera_link carried over
- gains.yaml regenerated (within 1 %); Isaac re-check: nominal 80/80, hard
  conditions pass at low stance only
- comms: second desktop->robot note (frames, L=+y, static lean, limits)

Co-Authored-By: Claude Opus 5.5 <noreply@anthropic.com>
Claude-Session: https://claude.ai/code/session_01UzDH5P8A4MBh8AMYdj2gqF

File: sim/model/robot_simple.urdf (robot description, URDF)
Before this commit: robot wheeled_biped_simple, 5 links, 4 joints
Links:
- removed link base
- added link base_link, mass 2.949467; collision box size=0.15 0.19 0.13; visual box size=0.15 0.19 0.13
- added link camera_link
- added link gps_link
- added link imu_link
- added link laser
- link l_carrier: mass 0.473631 -> 0.473474
- link r_carrier: mass 0.473631 -> 0.473474
Joints:
- added joint camera_link_joint: type fixed, parent base_link, child camera_link, origin xyz=0.107996 0 0.0152593 rpy=0 0 -0
- added joint gps_link_joint: type fixed, parent base_link, child gps_link, origin xyz=0.0503105 -0.004766 0.0863994 rpy=0 -0 -0
- added joint imu_link_joint: type fixed, parent base_link, child imu_link, origin xyz=0.0499964 -0.005 0.0699994 rpy=-0 -0 -0
- added joint laser_joint: type fixed, parent base_link, child laser, origin xyz=-0.0774261 0 0.122499 rpy=-0 -0 -3.14159
- joint l_leg: origin xyz=0 -0.081 0 rpy=0 0 0 -> xyz=0 0.081 0 rpy=0 0 0; parent base -> base_link
- joint r_leg: origin xyz=0 0.081 0 rpy=0 0 0 -> xyz=0 -0.081 0 rpy=0 0 0; parent base -> base_link
