Commit message: sim+docs+comms: 바퀴 실측 (휠 + 고무 72.5 g, 고무 16.5 g) — 총 4.170 kg, 바퀴 축 관성 2.681e-4 (메시 + 실측 질량), WHEEL_IZZ 1.8414e-3
- usd_loop = export 7 + 바퀴 실측 (usd_loop_e7 = export 7 그대로). 폐루프 잔차 0.00 mm, leg_map 0.02 mm
- pv harsh 98.9 % (실행마다 같음, export 7 바퀴 그대로 99.0 % — 차 7/4096), robust 11 종 x16 167/176
- harsh_eval 도 시작 때 모델 경로·총질량 출력
- 고무 30 g 추정 정정 (실측 16.5 g)

Co-Authored-By: Claude Opus 5.5 <noreply@anthropic.com>

File: sim/model/cad_export7_robot.urdf (robot description, URDF)
Before this commit: robot wheeled_biped_FIN, 21 links, 20 joints
Links:
- link l_wheel: mass 0.0701988 -> 0.0725
- link r_wheel: mass 0.0701988 -> 0.0725
