Commit message: sim: new wheel measured (hub 66 g + rubber 26 g = 92.0 g) — mesh-shaped inertia 3.363e-4, default model
- export_(8b): wheel mass 0.092, COM z -5.42 mm, izz 3.3633e-4 + rotor 1.5733e-3 = 1.9096e-3 (CAD 94.7 g: 1.9111e-3)
- usd_loop = 8b, usd_loop_e8 = CAD wheel; balance_tables.yaml regenerated (lqr_k change < 0.01 %)

Co-Authored-By: Claude Opus 5.5 <noreply@anthropic.com>
Claude-Session: https://claude.ai/code/session_01UzDH5P8A4MBh8AMYdj2gqF

File: sim/model/cad_export8_robot.urdf (robot description, URDF)
Before this commit: robot wheeled_biped_FIN_nwewheel, 21 links, 20 joints
Links:
- link l_wheel: mass 0.0946988 -> 0.092
- link r_wheel: mass 0.0946988 -> 0.092
